File: kicad/amper/amper.sch (KiCad schematic (older format))
At the start: 45 parts, among them J1 Conn_01x05, J2 Conn_01x02, J3 Conn_01x15, J4 Conn_01x10, J5 Conn_01x10, Q1 FDS9435A, Q2 FDS9435A, SW1 SW_Push, SW2 SW_Push, SW3 SW_Push, SW4 SW_Push, U1 TM1637, U2 HDSM-441B, U3 HDSM-441B, U4 HDSM-441B, U5 UA741CP, U6 ATtiny40-SU

Commit message: amper rev a
Parts:
- renumbered R3 to R1, R4 to R2, R1 to R3, R2 to R4, SW3 to SW1, SW4 to SW2, SW1 to SW3, SW2 to SW4, U5 to U1, U4 to U3, U3 to U4, U1 to U5
Connections:
- net at J2.1 (Pin_1): now also U1.3 (+); no longer U1.2 (-)
- net at J2.2 (Pin_2): now also U1.2 (-); no longer U1.3 (+)
Changed lines of the file:
@@
 $EndDescr
 $Comp
-L power:+5V #PWR0101
+L power:+5V #PWR03
 U 1 1 61CC1B88
 P 2700 4600
-F 0 "#PWR0101" H 2700 4450 50  0001 C CNN
+F 0 "#PWR03" H 2700 4450 50  0001 C CNN
 F 1 "+5V" H 2715 4773 50  0000 C CNN
 F 2 "" H 2700 4600 50  0001 C CNN
@@
 	3200 5000 3100 5000
 $Comp
-L power:GND #PWR0102
+L power:GND #PWR04
 U 1 1 61CDCA7A
 P 2700 5400
-F 0 "#PWR0102" H 2700 5150 50  0001 C CNN
+F 0 "#PWR04" H 2700 5150 50  0001 C CNN
 F 1 "GND" H 2705 5227 50  0000 C CNN
 F 2 "" H 2700 5400 50  0001 C CNN
@@
 	1    2700 5400
 	1    0    0    -1
-$EndComp
-$Comp
-L Connector_Generic:Conn_01x02 J2
-U 1 1 61CF2DA2
-P 2200 5050
-F 0 "J2" H 2118 4817 50  0000 C CNN
-F 1 "Conn_01x02" H 2118 4816 50  0001 C CNN
-F 2 "amper:2.54_2x5_row_ganged" H 2200 5050 50  0001 C CNN
-F 3 "~" H 2200 5050 50  0001 C CNN
-	1    2200 5050
-	-1   0    0    1
 $EndComp
 Wire Wire Line
@@
 	1550 4900 1650 4900
 $Comp
-L Display_Character:HDSM-441B U4
+L Display_Character:HDSM-441B U3
 U 1 1 61D03834
 P 3450 2350
-F 0 "U4" H 3450 2925 50  0000 C CNN
+F 0 "U3" H 3450 2925 50  0000 C CNN
 F 1 "HDSM-441B" H 3450 2926 50  0001 C CNN
 F 2 "amper:SLS0392FB4A1GD" H 3450 1750 50  0001 C CNN
@@
 	4050 1600 4150 1600
 $Comp
-L Switch:SW_Push SW3
+L Switch:SW_Push SW1
 U 1 1 61DB52EF
 P 1550 2300
-F 0 "SW3" H 1550 2585 50  0000 C CNN
+F 0 "SW1" H 1550 2585 50  0000 C CNN
 F 1 "SW_Push" H 1550 2494 50  0000 C CNN
 F 2 "amper:K2-1157SP-I4SW-01" H 1550 2500 50  0001 C CNN
@@
 $EndComp
 $Comp
-L Switch:SW_Push SW4
+L Switch:SW_Push SW2
 U 1 1 61DB52F5
 P 1550 2700
-F 0 "SW4" H 1550 2985 50  0000 C CNN
+F 0 "SW2" H 1550 2985 50  0000 C CNN
 F 1 "SW_Push" H 1550 2894 50  0000 C CNN
 F 2 "amper:K2-1157SP-I4SW-01" H 1550 2900 50  0001 C CNN
@@
 $EndComp
 $Comp
-L Device:R R3
+L Device:R R1
 U 1 1 61DB52FB
 P 2000 2300
-F 0 "R3" V 1793 2300 50  0000 C CNN
+F 0 "R1" V 1793 2300 50  0000 C CNN
 F 1 "10K" V 1884 2300 50  0000 C CNN
 F 2 "Resistor_SMD:R_0603_1608Metric_Pad1.05x0.95mm_HandSolder" V 1930 2300 50  0001 C CNN
@@
 $EndComp
 $Comp
-L power:+5V #PWR0104
+L power:+5V #PWR01
 U 1 1 61DB5301
 P 2250 2200
-F 0 "#PWR0104" H 2250 2050 50  0001 C CNN
+F 0 "#PWR01" H 2250 2050 50  0001 C CNN
 F 1 "+5V" H 2265 2373 50  0000 C CNN
 F 2 "" H 2250 2200 50  0001 C CNN
@@
 $EndComp
 $Comp
-L Device:R R4
+L Device:R R2
 U 1 1 61DB5307
 P 2000 2700
-F 0 "R4" V 1793 2700 50  0000 C CNN
+F 0 "R2" V 1793 2700 50  0000 C CNN
 F 1 "10K" V 1884 2700 50  0000 C CNN
 F 2 "Resistor_SMD:R_0603_1608Metric_Pad1.05x0.95mm_HandSolder" V 1930 2700 50  0001 C CNN
@@
 	2250 2300 2250 2200
 $Comp
-L amper-symbols:TM1637 U1
+L amper-symbols:TM1637 U5
 U 1 1 61DD858A
 P 4100 7050
-F 0 "U1" H 4100 7725 50  0000 C CNN
+F 0 "U5" H 4100 7725 50  0000 C CNN
 F 1 "TM1637" H 4100 7634 50  0000 C CNN
 F 2 "amper:TM1637" H 3750 7500 50  0001 C CNN
@@
 	3650 7400 3550 7400
 $Comp
-L power:GND #PWR0105
+L power:GND #PWR05
 U 1 1 61DDF936
 P 3150 6700
-F 0 "#PWR0105" H 3150 6450 50  0001 C CNN
+F 0 "#PWR05" H 3150 6450 50  0001 C CNN
 F 1 "GND" H 3155 6527 50  0000 C CNN
 F 2 "" H 3150 6700 50  0001 C CNN
@@
 	3650 7500 3550 7500
 $Comp
-L power:+5V #PWR0106
+L power:+5V #PWR010
 U 1 1 61DF9930
 P 6350 6900
-F 0 "#PWR0106" H 6350 6750 50  0001 C CNN
+F 0 "#PWR010" H 6350 6750 50  0001 C CNN
 F 1 "+5V" H 6365 7073 50  0000 C CNN
 F 2 "" H 6350 6900 50  0001 C CNN
@@
 	4550 7000 5000 7000
 $Comp
-L power:GND #PWR0107
+L power:GND #PWR011
 U 1 1 61E16664
 P 6600 6000
-F 0 "#PWR0107" H 6600 5750 50  0001 C CNN
+F 0 "#PWR011" H 6600 5750 50  0001 C CNN
 F 1 "GND" H 6605 5827 50  0000 C CNN
 F 2 "" H 6600 6000 50  0001 C CNN
@@
 	1750 3850 1850 3850
 $Comp
-L Device:R R2
+L Device:R R4
 U 1 1 61D581C2
 P 2000 3850
-F 0 "R2" V 1793 3850 50  0000 C CNN
+F 0 "R4" V 1793 3850 50  0000 C CNN
 F 1 "10K" V 1884 3850 50  0000 C CNN
 F 2 "Resistor_SMD:R_0603_1608Metric_Pad1.05x0.95mm_HandSolder" V 1930 3850 50  0001 C CNN
@@
 $EndComp
 $Comp
-L power:+5V #PWR0103
+L power:+5V #PWR02
 U 1 1 61D22891
 P 2250 3350
-F 0 "#PWR0103" H 2250 3200 50  0001 C CNN
+F 0 "#PWR02" H 2250 3200 50  0001 C CNN
 F 1 "+5V" H 2265 3523 50  0000 C CNN
 F 2 "" H 2250 3350 50  0001 C CNN
@@
 $EndComp
 $Comp
-L Device:R R1
+L Device:R R3
 U 1 1 61D22886
 P 2000 3450
-F 0 "R1" V 1793 3450 50  0000 C CNN
+F 0 "R3" V 1793 3450 50  0000 C CNN
 F 1 "10K" V 1884 3450 50  0000 C CNN
 F 2 "Resistor_SMD:R_0603_1608Metric_Pad1.05x0.95mm_HandSolder" V 1930 3450 50  0001 C CNN
@@
 SourceBUp
 $Comp
-L Switch:SW_Push SW2
+L Switch:SW_Push SW4
 U 1 1 61D2287E
 P 1550 3850
-F 0 "SW2" H 1550 4135 50  0000 C CNN
+F 0 "SW4" H 1550 4135 50  0000 C CNN
 F 1 "SW_Push" H 1550 4044 50  0000 C CNN
 F 2 "amper:K2-1157SP-I4SW-01" H 1550 4050 50  0001 C CNN
@@
 $EndComp
 $Comp
-L Switch:SW_Push SW1
+L Switch:SW_Push SW3
 U 1 1 61D22878
 P 1550 3450
-F 0 "SW1" H 1550 3735 50  0000 C CNN
+F 0 "SW3" H 1550 3735 50  0000 C CNN
 F 1 "SW_Push" H 1550 3644 50  0000 C CNN
 F 2 "amper:K2-1157SP-I4SW-01" H 1550 3650 50  0001 C CNN
@@
 SEG1
 $Comp
-L Display_Character:HDSM-441B U3
+L Display_Character:HDSM-441B U4
 U 1 1 61D2285E
 P 3450 3500
-F 0 "U3" H 3450 4075 50  0000 C CNN
+F 0 "U4" H 3450 4075 50  0000 C CNN
 F 1 "HDSM-441B" H 3450 4076 50  0001 C CNN
 F 2 "amper:SLS0392FB4A1GD" H 3450 2900 50  0001 C CNN
@@
 	6000 3150 6000 3050
 $Comp
-L power:+5V #PWR0108
+L power:+5V #PWR08
 U 1 1 61EFA68D
 P 6000 3050
-F 0 "#PWR0108" H 6000 2900 50  0001 C CNN
+F 0 "#PWR08" H 6000 2900 50  0001 C CNN
 F 1 "+5V" H 6015 3223 50  0000 C CNN
 F 2 "" H 6000 3050 50  0001 C CNN
@@
 Connection ~ 6000 4150
 $Comp
-L power:GND #PWR0109
+L power:GND #PWR09
 U 1 1 61EFA69E
 P 6000 4250
-F 0 "#PWR0109" H 6000 4000 50  0001 C CNN
+F 0 "#PWR09" H 6000 4000 50  0001 C CNN
 F 1 "GND" H 6005 4077 50  0000 C CNN
 F 2 "" H 6000 4250 50  0001 C CNN
@@
 $EndComp
 $Comp
-L power:+5V #PWR0110
+L power:+5V #PWR012
 U 1 1 62001D6A
 P 9200 5550
-F 0 "#PWR0110" H 9200 5400 50  0001 C CNN
+F 0 "#PWR012" H 9200 5400 50  0001 C CNN
 F 1 "+5V" H 9215 5723 50  0000 C CNN
 F 2 "" H 9200 5550 50  0001 C CNN
@@
 Connection ~ 9200 5650
 $Comp
-L power:GND #PWR0111
+L power:GND #PWR013
 U 1 1 62050EDB
 P 9200 6050
-F 0 "#PWR0111" H 9200 5800 50  0001 C CNN
+F 0 "#PWR013" H 9200 5800 50  0001 C CNN
 F 1 "GND" H 9205 5877 50  0000 C CNN
 F 2 "" H 9200 6050 50  0001 C CNN
@@
 	5950 1000 5950 900
 $Comp
-L power:+5V #PWR0112
+L power:+5V #PWR06
 U 1 1 621F0C2E
 P 5950 900
-F 0 "#PWR0112" H 5950 750 50  0001 C CNN
+F 0 "#PWR06" H 5950 750 50  0001 C CNN
 F 1 "+5V" H 5965 1073 50  0000 C CNN
 F 2 "" H 5950 900 50  0001 C CNN
@@
 Connection ~ 5950 2000
 $Comp
-L power:GND #PWR0113
+L power:GND #PWR07
 U 1 1 621F0C3E
 P 5950 2100
-F 0 "#PWR0113" H 5950 1850 50  0001 C CNN
+F 0 "#PWR07" H 5950 1850 50  0001 C CNN
 F 1 "GND" H 5955 1927 50  0000 C CNN
 F 2 "" H 5950 2100 50  0001 C CNN
@@
 	7450 2100 7450 2500
 $Comp
-L Amplifier_Operational:LM741 U5
+L Amplifier_Operational:LM741 U1
 U 1 1 62259D5D
 P 2800 5000
-F 0 "U5" H 2800 5250 50  0000 L CNN
+F 0 "U1" H 2800 5250 50  0000 L CNN
 F 1 "UA741CP" H 2850 5150 50  0000 L CNN
 F 2 "amper:114-87-308-41-134161" H 2850 5050 50  0001 C CNN
@@
 	1    0    0    -1
 $EndComp
+$Comp
+L Connector_Generic:Conn_01x02 J2
+U 1 1 61CF2DA2
+P 2200 4950
+F 0 "J2" H 2118 4717 50  0000 C CNN
+F 1 "Conn_01x02" H 2118 4716 50  0001 C CNN
+F 2 "amper:2.54_2x5_row_ganged" H 2200 4950 50  0001 C CNN
+F 3 "~" H 2200 4950 50  0001 C CNN
+	1    2200 4950
+	-1   0    0    -1
+$EndComp
 $EndSCHEMATC

Commit message: Amper rev A ready to go
Parts:
- added U7: UA741CP, symbol Amplifier_Operational:LM741
- C1, C2, C3, C5, C6, C7, C8, R1, R10, R11, R12, R13, R14, R2, R3, R4, R5, R6, R7, R8, R9: Vendor (none) -> Already Have
- C4: Part (none) -> C85713; Vendor (none) -> LCSC
- J1, J2: Part (none) -> C843271; Vendor (none) -> LCSC
- J3, J4, J5, TP1, TP2, TP3, TP4, TP5, TP6: Vendor (none) -> Do Not Fit
- Q1, Q2: Part (none) -> C181098; Vendor (none) -> LCSC
- SW1, SW2, SW3, SW4: Part (none) -> C2909692; Vendor (none) -> LCSC
- U1: value UA741CP -> 114-87-308-41-134161; Vendor (none) -> Not LCSC
- U2, U3, U4: Part (none) -> C226000; Vendor (none) -> LCSC
- U5: Part (none) -> C20001; Vendor (none) -> LCSC
- U6: Vendor (none) -> Not LCSC
Connections:
- no-connect marks 4 -> 11

Commit message: added easy fixes from testing to sch
Parts:
- added C? (x2): 5uF, symbol Device:CP1
- C4: value 10uF -> 2uF
- R10, R12: value 40k -> 20k
- R11, R9: value 25k -> 12k
- R7, R8: value 60k -> 30k
Connections:
- net +5V: now also Q1.1 (S), Q1.2 (S), Q1.3 (S), Q2.1 (S), Q2.2 (S), Q2.3 (S); no longer Q1.5 (D), Q1.6 (D), Q1.7 (D), Q1.8 (D), Q2.5 (D), Q2.6 (D), Q2.7 (D), Q2.8 (D)
- net GND: now also C?.2, C?.2
- net SourceA: now also Q1.5 (D), Q1.6 (D), Q1.7 (D), Q1.8 (D), C?.1; no longer Q1.1 (S), Q1.2 (S), Q1.3 (S)
- net SourceB: now also Q2.5 (D), Q2.6 (D), Q2.7 (D), Q2.8 (D), C?.1; no longer Q2.1 (S), Q2.2 (S), Q2.3 (S)
Other:
- note added: "Determine\ncombination\nwith testing"
Changed lines of the file:
@@
 P 6100 6150
 F 0 "C4" H 6215 6196 50  0000 L CNN
-F 1 "10uF" H 6100 6050 50  0000 L CNN
+F 1 "2uF" H 6100 6050 50  0000 L CNN
 F 2 "Capacitor_SMD:C_0603_1608Metric_Pad1.05x0.95mm_HandSolder" H 6138 6000 50  0001 C CNN
 F 3 "~" H 6100 6150 50  0001 C CNN
@@
 Wire Wire Line
 	7400 1900 7400 2000
-Wire Wire Line
-	7400 1550 7500 1550
-Text Label 7500 1550 0    50   ~ 0
+Text Label 7900 1550 0    50   ~ 0
 SourceA
 Wire Wire Line
@@
 P 5750 3650
 F 0 "R8" V 5543 3650 50  0000 C CNN
-F 1 "60k" V 5634 3650 50  0000 C CNN
+F 1 "30k" V 5634 3650 50  0000 C CNN
 F 2 "Resistor_SMD:R_0603_1608Metric_Pad1.05x0.95mm_HandSolder" V 5680 3650 50  0001 C CNN
 F 3 "~" H 5750 3650 50  0001 C CNN
@@
 P 6000 3400
 F 0 "R11" H 6070 3446 50  0000 L CNN
-F 1 "25k" H 6070 3355 50  0000 L CNN
+F 1 "12k" H 6070 3355 50  0000 L CNN
 F 2 "Resistor_SMD:R_0603_1608Metric_Pad1.05x0.95mm_HandSolder" V 5930 3400 50  0001 C CNN
 F 3 "~" H 6000 3400 50  0001 C CNN
@@
 P 6000 3900
 F 0 "R12" H 6070 3946 50  0000 L CNN
-F 1 "40k" H 6070 3855 50  0000 L CNN
+F 1 "20k" H 6070 3855 50  0000 L CNN
 F 2 "Resistor_SMD:R_0603_1608Metric_Pad1.05x0.95mm_HandSolder" V 5930 3900 50  0001 C CNN
 F 3 "~" H 6000 3900 50  0001 C CNN
@@
 Wire Wire Line
 	6600 3450 6700 3450
-Wire Wire Line
-	7450 3700 7550 3700
-Text Label 7550 3700 0    50   ~ 0
+Text Label 7950 3700 0    50   ~ 0
 SourceB
 $Comp
@@
 This resistor may be\nuneccassary depending\non open circuit drain\ntime
 Wire Notes Line
-	6900 3750 7300 3750
-Wire Notes Line
 	7300 3750 7300 4250
 Wire Notes Line
 	7500 4250 7500 4650
-Wire Notes Line
-	7500 4650 6550 4650
 Wire Notes Line
 	6550 4650 6550 4250
@@
 P 5700 1500
 F 0 "R7" V 5493 1500 50  0000 C CNN
-F 1 "60k" V 5584 1500 50  0000 C CNN
+F 1 "30k" V 5584 1500 50  0000 C CNN
 F 2 "Resistor_SMD:R_0603_1608Metric_Pad1.05x0.95mm_HandSolder" V 5630 1500 50  0001 C CNN
 F 3 "~" H 5700 1500 50  0001 C CNN
@@
 P 5950 1250
 F 0 "R9" H 6020 1296 50  0000 L CNN
-F 1 "25k" H 6020 1205 50  0000 L CNN
+F 1 "12k" H 6020 1205 50  0000 L CNN
 F 2 "Resistor_SMD:R_0603_1608Metric_Pad1.05x0.95mm_HandSolder" V 5880 1250 50  0001 C CNN
 F 3 "~" H 5950 1250 50  0001 C CNN
@@
 P 5950 1750
 F 0 "R10" H 6020 1796 50  0000 L CNN
-F 1 "40k" H 6020 1705 50  0000 L CNN
+F 1 "20k" H 6020 1705 50  0000 L CNN
 F 2 "Resistor_SMD:R_0603_1608Metric_Pad1.05x0.95mm_HandSolder" V 5880 1750 50  0001 C CNN
 F 3 "~" H 5950 1750 50  0001 C CNN
@@
 This resistor may be\nuneccassary depending\non open circuit drain\ntime
 Wire Notes Line
-	6850 1600 7250 1600
-Wire Notes Line
 	7250 1600 7250 2100
-Wire Notes Line
-	7450 2500 6500 2500
 Wire Notes Line
 	6500 2500 6500 2100
@@
 F 5 "C181098" H 6900 3450 50  0001 C CNN "Part"
 	1    6900 3450
-	1    0    0    -1
+	1    0    0    1
 $EndComp
 $Comp
@@
 F 5 "C181098" H 6850 1300 50  0001 C CNN "Part"
 	1    6850 1300
-	1    0    0    -1
+	1    0    0    1
 $EndComp
 $Comp
@@
 	1    0    0    -1
 $EndComp
+$Comp
+L Device:CP1 C?
+U 1 1 62175534
+P 7850 3900
+F 0 "C?" H 7965 3946 50  0000 L CNN
+F 1 "5uF" H 7965 3855 50  0000 L CNN
+F 2 "" H 7850 3900 50  0001 C CNN
+F 3 "~" H 7850 3900 50  0001 C CNN
+	1    7850 3900
+	1    0    0    -1
+$EndComp
+Wire Wire Line
+	7450 4150 7850 4150
+Wire Wire Line
+	7850 4150 7850 4050
+Connection ~ 7450 4150
+Wire Wire Line
+	7450 3700 7850 3700
+Wire Wire Line
+	7850 3750 7850 3700
+Connection ~ 7850 3700
+Wire Wire Line
+	7850 3700 7950 3700
+Wire Notes Line
+	8200 3750 8200 4650
+Wire Notes Line
+	6900 3750 8200 3750
+Wire Notes Line
+	6550 4650 8200 4650
+Text Notes 7650 4500 0    50   ~ 0
+Determine\ncombination\nwith testing
+$Comp
+L Device:CP1 C?
+U 1 1 621C95BD
+P 7800 1750
+F 0 "C?" H 7915 1796 50  0000 L CNN
+F 1 "5uF" H 7915 1705 50  0000 L CNN
+F 2 "" H 7800 1750 50  0001 C CNN
+F 3 "~" H 7800 1750 50  0001 C CNN
+	1    7800 1750
+	1    0    0    -1
+$EndComp
+Wire Wire Line
+	7400 2000 7800 2000
+Wire Wire Line
+	7800 2000 7800 1900
+Text Notes 7600 2350 0    50   ~ 0
+Determine\ncombination\nwith testing
+Wire Notes Line
+	6500 2500 8150 2500
+Wire Wire Line
+	7400 1550 7800 1550
+Wire Wire Line
+	7800 1600 7800 1550
+Connection ~ 7800 1550
+Wire Wire Line
+	7800 1550 7900 1550
+Wire Notes Line
+	8150 1600 8150 2500
+Wire Notes Line
+	6850 1600 8150 1600
 $EndSCHEMATC

Commit message: added attiny1606
Parts:
- removed U6: ATtiny40-SU, Package_SO:SOIC-20W_7.5x12.8mm_P1.27mm, symbol MCU_Microchip_ATtiny:ATtiny40-SU
- added U?: ATtiny1606-S, Package_SO:SOIC-20W_7.5x12.8mm_P1.27mm, symbol amper-symbols:ATtiny1606-S
Connections:
- net +5V: now also J4.1 (Pin_1), U?.1 (VCC)
- net GND: now also J5.10 (Pin_10), U?.20 (GND)
- net at J4.10 (Pin_10): now also U?.10 (PB1)
- net at J5.1 (Pin_1): now also U?.11 (PB0)
- net at J5.2 (Pin_2): now also U?.12 (PC0)
- net at J5.3 (Pin_3): now also U?.13 (PC1)
- net at J5.4 (Pin_4): now also U?.14 (PC2)
- net at J5.5 (Pin_5): now also U?.15 (PC3)
- net at J5.6 (Pin_6): now also U?.16 (~RESET~/PA0)
- net at J5.7 (Pin_7): now also U?.17 (PA1)
- net at J5.8 (Pin_8): now also U?.18 (PA2)
- net at J5.9 (Pin_9): now also U?.19 (PA3)
- net at J4.2 (Pin_2): now also U?.2 (PA4)
- net at J4.3 (Pin_3): now also U?.3 (PA5)
- net at J4.4 (Pin_4): now also U?.4 (PA6)
- net at J4.5 (Pin_5): now also U?.5 (PA7)
- net at J4.6 (Pin_6): now also U?.6 (PB5)
- net at J4.7 (Pin_7): now also U?.7 (PB4)
- net at J4.8 (Pin_8): now also U?.8 (PB3)
- net at J4.9 (Pin_9): now also U?.9 (PB2)
Other:
- moved on the sheet: J4, J5
Changed lines of the file:
@@
 	5550 3100 5550 4100
-$Comp
-L MCU_Microchip_ATtiny:ATtiny40-SU U6
-U 1 1 61F15A5A
-P 9500 2600
-F 0 "U6" H 8970 2646 50  0000 R CNN
-F 1 "ATtiny40-SU" H 8970 2555 50  0000 R CNN
-F 2 "Package_SO:SOIC-20W_7.5x12.8mm_P1.27mm" H 9500 2600 50  0001 C CIN
-F 3 "~" H 9500 2600 50  0001 C CNN
-F 4 "Not LCSC" H 9500 2600 50  0001 C CNN "Vendor"
-	1    9500 2600
-	1    0    0    -1
-$EndComp
 $Comp
 L Connector_Generic:Conn_01x10 J4
 U 1 1 61F3370B
-P 10700 2000
-F 0 "J4" H 10618 1275 50  0000 C CNN
-F 1 "Conn_01x10" H 10618 1366 50  0000 C CNN
-F 2 "Connector_PinSocket_2.54mm:PinSocket_1x10_P2.54mm_Vertical" H 10700 2000 50  0001 C CNN
-F 3 "~" H 10700 2000 50  0001 C CNN
-F 4 "Do Not Fit" H 10700 2000 50  0001 C CNN "Vendor"
-	1    10700 2000
-	1    0    0    1
-$EndComp
-Wire Wire Line
-	10100 1600 10500 1600
-Wire Wire Line
-	10100 1700 10500 1700
-Wire Wire Line
-	10100 1800 10500 1800
-Wire Wire Line
-	10100 1900 10500 1900
-Wire Wire Line
-	10100 2000 10500 2000
-Wire Wire Line
-	10100 2100 10500 2100
-Wire Wire Line
-	10100 2200 10500 2200
-Wire Wire Line
-	10100 2300 10500 2300
-Wire Wire Line
-	10100 2500 10300 2500
-Wire Wire Line
-	10300 2500 10300 2400
-Wire Wire Line
-	10300 2400 10500 2400
+P 8550 2850
+F 0 "J4" H 8468 2125 50  0000 C CNN
+F 1 "Conn_01x10" H 8468 2216 50  0000 C CNN
+F 2 "Connector_PinSocket_2.54mm:PinSocket_1x10_P2.54mm_Vertical" H 8550 2850 50  0001 C CNN
+F 3 "~" H 8550 2850 50  0001 C CNN
+F 4 "Do Not Fit" H 8550 2850 50  0001 C CNN "Vendor"
+	1    8550 2850
+	-1   0    0    -1
+$EndComp
 $Comp
 L Connector_Generic:Conn_01x10 J5
 U 1 1 61F743AC
-P 10700 3200
-F 0 "J5" H 10618 2475 50  0000 C CNN
-F 1 "Conn_01x10" H 10618 2566 50  0000 C CNN
-F 2 "Connector_PinSocket_2.54mm:PinSocket_1x10_P2.54mm_Vertical" H 10700 3200 50  0001 C CNN
-F 3 "~" H 10700 3200 50  0001 C CNN
-F 4 "Do Not Fit" H 10700 3200 50  0001 C CNN "Vendor"
-	1    10700 3200
+P 10850 2950
+F 0 "J5" H 10768 2225 50  0000 C CNN
+F 1 "Conn_01x10" H 10768 2316 50  0000 C CNN
+F 2 "Connector_PinSocket_2.54mm:PinSocket_1x10_P2.54mm_Vertical" H 10850 2950 50  0001 C CNN
+F 3 "~" H 10850 2950 50  0001 C CNN
+F 4 "Do Not Fit" H 10850 2950 50  0001 C CNN "Vendor"
+	1    10850 2950
 	1    0    0    1
 $EndComp
-Wire Wire Line
-	10100 3000 10500 3000
-Wire Wire Line
-	10100 3100 10500 3100
-Wire Wire Line
-	10100 3200 10500 3200
-Wire Wire Line
-	10100 3300 10500 3300
-Wire Wire Line
-	10100 3400 10500 3400
-Wire Wire Line
-	10100 3500 10500 3500
-Wire Wire Line
-	10500 2900 10200 2900
-Wire Wire Line
-	10200 2900 10200 2800
-Wire Wire Line
-	10200 2800 10100 2800
-Wire Wire Line
-	10100 2700 10300 2700
-Wire Wire Line
-	10300 2700 10300 2800
-Wire Wire Line
-	10300 2800 10500 2800
-Wire Wire Line
-	10400 2600 10400 2700
-Wire Wire Line
-	10400 2700 10500 2700
-Wire Wire Line
-	10100 2600 10400 2600
-Wire Wire Line
-	10500 1500 10300 1500
-Wire Wire Line
-	10300 1500 10300 1150
-Wire Wire Line
-	10300 1150 10900 1150
-Wire Wire Line
-	10900 1150 10900 4050
-Wire Wire Line
-	10900 4050 9500 4050
-Wire Wire Line
-	9500 4050 9500 3900
-Wire Wire Line
-	10500 3600 10350 3600
-Wire Wire Line
-	10350 3600 10350 4150
-Wire Wire Line
-	10350 4150 8400 4150
-Wire Wire Line
-	8400 4150 8400 1200
-Wire Wire Line
-	8400 1200 9500 1200
-Wire Wire Line
-	9500 1200 9500 1300
 Text Label 9850 4550 2    50   ~ 0
 CLK
@@
 Wire Notes Line
 	6850 1600 8150 1600
+$Comp
+L amper-symbols:ATtiny1606-S U?
+U 1 1 62224E78
+P 9700 3150
+F 0 "U?" H 9700 4115 50  0000 C CNN
+F 1 "ATtiny1606-S" H 9700 4024 50  0000 C CNN
+F 2 "Package_SO:SOIC-20W_7.5x12.8mm_P1.27mm" H 9700 2800 50  0001 C CIN
+F 3 "http://ww1.microchip.com/downloads/en/DeviceDoc/ATtiny806_1606_Data_Sheet_40002029A.pdf" H 9700 3150 50  0001 C CNN
+	1    9700 3150
+	1    0    0    -1
+$EndComp
+Wire Wire Line
+	8750 2450 9000 2450
+Wire Wire Line
+	8750 2550 9100 2550
+Wire Wire Line
+	8750 2650 9100 2650
+Wire Wire Line
+	8750 2750 9100 2750
+Wire Wire Line
+	8750 2850 9100 2850
+Wire Wire Line
+	8750 2950 9100 2950
+Wire Wire Line
+	8750 3050 9100 3050
+Wire Wire Line
+	8750 3150 9100 3150
+Wire Wire Line
+	8750 3250 9100 3250
+Wire Wire Line
+	8750 3350 9100 3350
+Wire Wire Line
+	10300 2450 10400 2450
+Wire Wire Line
+	10300 2550 10650 2550
+Wire Wire Line
+	10300 2650 10650 2650
+Wire Wire Line
+	10300 2750 10650 2750
+Wire Wire Line
+	10300 2850 10650 2850
+Wire Wire Line
+	10300 2950 10650 2950
+Wire Wire Line
+	10300 3050 10650 3050
+Wire Wire Line
+	10300 3150 10650 3150
+Wire Wire Line
+	10300 3250 10650 3250
+Wire Wire Line
+	10300 3350 10650 3350
+$Comp
+L power:+5V #PWR?
+U 1 1 622DD6E8
+P 9000 2350
+F 0 "#PWR?" H 9000 2200 50  0001 C CNN
+F 1 "+5V" H 9015 2523 50  0000 C CNN
+F 2 "" H 9000 2350 50  0001 C CNN
+F 3 "" H 9000 2350 50  0001 C CNN
+	1    9000 2350
+	1    0    0    -1
+$EndComp
+Wire Wire Line
+	9000 2350 9000 2450
+Connection ~ 9000 2450
+Wire Wire Line
+	9000 2450 9100 2450
+$Comp
+L power:GND #PWR?
+U 1 1 622EC3F9
+P 10150 2100
+F 0 "#PWR?" H 10150 1850 50  0001 C CNN
+F 1 "GND" H 10155 1927 50  0000 C CNN
+F 2 "" H 10150 2100 50  0001 C CNN
+F 3 "" H 10150 2100 50  0001 C CNN
+	1    10150 2100
+	1    0    0    -1
+$EndComp
+Wire Wire Line
+	10400 2450 10400 2000
+Wire Wire Line
+	10400 2000 10150 2000
+Wire Wire Line
+	10150 2000 10150 2100
+Connection ~ 10400 2450
+Wire Wire Line
+	10400 2450 10650 2450
 $EndSCHEMATC

Commit message: netlist rename pass
Connections:
- net AmpOut renamed ResultAdc
- net CLK renamed Tm1636Clk
- net DIO renamed Tm1636Dio
- net SourceA renamed SourceAAdc
- net SourceAPWM renamed SourceAPwm
- net SourceB renamed SourceBAdc
- net SourceBPWM renamed SourceBPwm
Changed lines of the file:
@@
 	1150 5000 1150 5650
 Text Label 1550 5100 2    50   ~ 0
-SourceA
+SourceAAdc
 Wire Wire Line
 	1550 5100 1650 5100
 Text Label 1550 4900 2    50   ~ 0
-SourceB
+SourceBAdc
 Wire Wire Line
 	1550 4900 1650 4900
@@
 	5300 5900 5000 5900
 Text Label 5500 6500 0    50   ~ 0
-DIO
+Tm1636Dio
 Text Label 5500 6400 0    50   ~ 0
-CLK
+Tm1636Clk
 $Comp
 L Device:C C3
@@
 Connection ~ 6100 7000
 Text Label 5350 1500 2    50   ~ 0
-SourceAPWM
+SourceAPwm
 Wire Wire Line
 	7400 1900 7400 2000
 Text Label 7900 1550 0    50   ~ 0
-SourceA
+SourceAAdc
 Wire Wire Line
 	2250 3450 2250 3350
@@
 	7400 1300 7400 1550
 Text Label 5400 3650 2    50   ~ 0
-SourceBPWM
+SourceBPwm
 $Comp
 L Device:R R8
@@
 	6600 3450 6700 3450
 Text Label 7950 3700 0    50   ~ 0
-SourceB
+SourceBAdc
 $Comp
 L Connector:TestPoint TP2
@@
 $EndComp
 Text Label 9850 4550 2    50   ~ 0
-CLK
+Tm1636Clk
 Text Label 9850 4650 2    50   ~ 0
-DIO
+Tm1636Dio
 Text Label 9850 4750 2    50   ~ 0
 SourceAUp
@@
 	9850 5050 9950 5050
 Text Label 3300 5000 0    50   ~ 0
-AmpOut
+ResultAdc
 Wire Wire Line
 	3300 5000 3200 5000
 Connection ~ 3200 5000
 Text Label 9850 5150 2    50   ~ 0
-SourceAPWM
+SourceAPwm
 Text Label 9850 5250 2    50   ~ 0
-SourceA
+SourceAAdc
 Text Label 9850 5350 2    50   ~ 0
-SourceBPWM
+SourceBPwm
 Text Label 9850 5450 2    50   ~ 0
-SourceB
+SourceBAdc
 Text Label 9850 5550 2    50   ~ 0
-AmpOut
+ResultAdc
 Wire Wire Line
 	9850 5150 9950 5150
