File: kicad/amper/amper.sch (KiCad schematic (older format))
At the start: 48 parts, among them J1 Conn_01x05, J2 Conn_01x02, J3 Conn_01x15, J4 Conn_01x10, J5 Conn_01x10, Q1 FDS9435A, Q2 FDS9435A, SW1 SW_Push, SW2 SW_Push, SW3 SW_Push, SW4 SW_Push, U1 114-87-308-41-134161, U2 HDSM-441B, U3 HDSM-441B, U4 HDSM-441B, U5 TM1637, U7 UA741CP

Commit message: added all connections from Amper 1606 port assignment in GDrive
Connections:
- net ResultAdc: now also J4.4 (Pin_4), U?.4 (PA6)
- net SourceAAdc: now also J5.7 (Pin_7), U?.17 (PA1)
- net SourceADn: now also J5.3 (Pin_3), U?.13 (PC1)
- net SourceAPwm: now also J5.9 (Pin_9), U?.19 (PA3)
- net SourceAUp: now also J5.2 (Pin_2), U?.12 (PC0)
- net SourceBAdc: now also J5.8 (Pin_8), U?.18 (PA2)
- net SourceBDn: now also J5.5 (Pin_5), U?.15 (PC3)
- net SourceBPwm: now also J5.1 (Pin_1), U?.11 (PB0)
- net SourceBUp: now also J5.4 (Pin_4), U?.14 (PC2)
- net Tm1637Clk: now reaches J4.2 (Pin_2), U?.2 (PA4)
- net Tm1637Dio: now reaches J4.3 (Pin_3), U?.3 (PA5)
- net UartRx: now reaches J4.8 (Pin_8), U?.8 (PB3)
- net UartTx: now reaches J4.9 (Pin_9), U?.9 (PB2)
- net AtProg: now reaches J5.6 (Pin_6), U?.16 (~RESET~/PA0)
Other:
- moved on the sheet: J4, J5
Changed lines of the file:
@@
 L Connector_Generic:Conn_01x10 J4
 U 1 1 61F3370B
-P 8550 2850
-F 0 "J4" H 8468 2125 50  0000 C CNN
-F 1 "Conn_01x10" H 8468 2216 50  0000 C CNN
-F 2 "Connector_PinSocket_2.54mm:PinSocket_1x10_P2.54mm_Vertical" H 8550 2850 50  0001 C CNN
-F 3 "~" H 8550 2850 50  0001 C CNN
-F 4 "Do Not Fit" H 8550 2850 50  0001 C CNN "Vendor"
-	1    8550 2850
+P 8400 2850
+F 0 "J4" H 8318 2125 50  0000 C CNN
+F 1 "Conn_01x10" H 8318 2216 50  0000 C CNN
+F 2 "Connector_PinSocket_2.54mm:PinSocket_1x10_P2.54mm_Vertical" H 8400 2850 50  0001 C CNN
+F 3 "~" H 8400 2850 50  0001 C CNN
+F 4 "Do Not Fit" H 8400 2850 50  0001 C CNN "Vendor"
+	1    8400 2850
 	-1   0    0    -1
 $EndComp
@@
 L Connector_Generic:Conn_01x10 J5
 U 1 1 61F743AC
-P 10850 2950
-F 0 "J5" H 10768 2225 50  0000 C CNN
-F 1 "Conn_01x10" H 10768 2316 50  0000 C CNN
-F 2 "Connector_PinSocket_2.54mm:PinSocket_1x10_P2.54mm_Vertical" H 10850 2950 50  0001 C CNN
-F 3 "~" H 10850 2950 50  0001 C CNN
-F 4 "Do Not Fit" H 10850 2950 50  0001 C CNN "Vendor"
-	1    10850 2950
+P 11000 2950
+F 0 "J5" H 10918 2225 50  0000 C CNN
+F 1 "Conn_01x10" H 10918 2316 50  0000 C CNN
+F 2 "Connector_PinSocket_2.54mm:PinSocket_1x10_P2.54mm_Vertical" H 11000 2950 50  0001 C CNN
+F 3 "~" H 11000 2950 50  0001 C CNN
+F 4 "Do Not Fit" H 11000 2950 50  0001 C CNN "Vendor"
+	1    11000 2950
 	1    0    0    1
 $EndComp
@@
 $EndComp
 Wire Wire Line
-	8750 2450 9000 2450
-Wire Wire Line
-	8750 2550 9100 2550
-Wire Wire Line
-	8750 2650 9100 2650
-Wire Wire Line
-	8750 2750 9100 2750
-Wire Wire Line
-	8750 2850 9100 2850
-Wire Wire Line
-	8750 2950 9100 2950
-Wire Wire Line
-	8750 3050 9100 3050
-Wire Wire Line
-	8750 3150 9100 3150
-Wire Wire Line
-	8750 3250 9100 3250
-Wire Wire Line
-	8750 3350 9100 3350
-Wire Wire Line
 	10300 2450 10400 2450
-Wire Wire Line
-	10300 2550 10650 2550
-Wire Wire Line
-	10300 2650 10650 2650
-Wire Wire Line
-	10300 2750 10650 2750
-Wire Wire Line
-	10300 2850 10650 2850
-Wire Wire Line
-	10300 2950 10650 2950
-Wire Wire Line
-	10300 3050 10650 3050
-Wire Wire Line
-	10300 3150 10650 3150
-Wire Wire Line
-	10300 3250 10650 3250
-Wire Wire Line
-	10300 3350 10650 3350
 $Comp
 L power:+5V #PWR?
@@
 	10150 2000 10150 2100
 Connection ~ 10400 2450
-Wire Wire Line
-	10400 2450 10650 2450
+Text Label 10350 2850 0    50   ~ 0
+AtProg
+Text Label 10350 2750 0    50   ~ 0
+SourceAAdc
+Wire Wire Line
+	10400 2450 10800 2450
+Wire Wire Line
+	10300 2550 10800 2550
+Wire Wire Line
+	10300 2650 10800 2650
+Wire Wire Line
+	10300 2750 10800 2750
+Wire Wire Line
+	10300 2850 10800 2850
+Wire Wire Line
+	10300 2950 10800 2950
+Wire Wire Line
+	10300 3050 10800 3050
+Wire Wire Line
+	10300 3150 10800 3150
+Wire Wire Line
+	10300 3250 10800 3250
+Wire Wire Line
+	10300 3350 10800 3350
+Text Label 10350 2650 0    50   ~ 0
+SourceBAdc
+Text Label 10350 2550 0    50   ~ 0
+SourceAPwm
+Text Label 9050 2550 2    50   ~ 0
+Tm1637Clk
+Wire Wire Line
+	8600 3350 9100 3350
+Wire Wire Line
+	8600 3250 9100 3250
+Wire Wire Line
+	8600 3050 9100 3050
+Wire Wire Line
+	8600 3150 9100 3150
+Wire Wire Line
+	8600 2850 9100 2850
+Wire Wire Line
+	8600 2950 9100 2950
+Wire Wire Line
+	8600 2650 9100 2650
+Wire Wire Line
+	8600 2750 9100 2750
+Wire Wire Line
+	8600 2450 9000 2450
+Wire Wire Line
+	8600 2550 9100 2550
+Text Label 9050 2650 2    50   ~ 0
+Tm1637Dio
+Text Label 9050 2750 2    50   ~ 0
+ResultAdc
+Text Label 10350 3350 0    50   ~ 0
+SourceBPwm
+Text Label 9000 3250 2    50   ~ 0
+UartTx
+Text Label 9000 3150 2    50   ~ 0
+UartRx
+Text Label 10350 3250 0    50   ~ 0
+SourceAUp
+Text Label 10350 3150 0    50   ~ 0
+SourceADn
+Text Label 10350 3050 0    50   ~ 0
+SourceBUp
+Text Label 10350 2950 0    50   ~ 0
+SourceBDn
 $EndSCHEMATC

Commit message: added breakout headers
Parts:
- added J6: Conn_01x03, amper:PROG, symbol Connector_Generic:Conn_01x03
- added J7: Conn_01x04, amper:UART, symbol Connector_Generic:Conn_01x04
- gave numbers to parts that had none: 3
Connections:
- net +5V: now also J6.1 (Pin_1), J7.1 (Pin_1)
- net AtProg: now also J6.2 (Pin_2)
- net GND: now also J6.3 (Pin_3), J7.4 (Pin_4)
- net UartRx: now also J7.3 (Pin_3)
- net UartTx: now also J7.2 (Pin_2)
Other:
- moved on the sheet: J3
Changed lines of the file:
@@
 	1    0    0    1
 $EndComp
-Text Label 9850 4550 2    50   ~ 0
+Text Label 8950 4600 2    50   ~ 0
 Tm1636Clk
-Text Label 9850 4650 2    50   ~ 0
+Text Label 8950 4700 2    50   ~ 0
 Tm1636Dio
-Text Label 9850 4750 2    50   ~ 0
+Text Label 8950 4800 2    50   ~ 0
 SourceAUp
-Text Label 9850 4850 2    50   ~ 0
+Text Label 8950 4900 2    50   ~ 0
 SourceADn
-Text Label 9850 4950 2    50   ~ 0
+Text Label 8950 5000 2    50   ~ 0
 SourceBUp
-Text Label 9850 5050 2    50   ~ 0
+Text Label 8950 5100 2    50   ~ 0
 SourceBDn
 Wire Wire Line
-	9850 4550 9950 4550
-Wire Wire Line
-	9850 4650 9950 4650
-Wire Wire Line
-	9850 4750 9950 4750
-Wire Wire Line
-	9850 4850 9950 4850
-Wire Wire Line
-	9850 4950 9950 4950
-Wire Wire Line
-	9850 5050 9950 5050
+	8950 4600 9050 4600
+Wire Wire Line
+	8950 4700 9050 4700
+Wire Wire Line
+	8950 4800 9050 4800
+Wire Wire Line
+	8950 4900 9050 4900
+Wire Wire Line
+	8950 5000 9050 5000
+Wire Wire Line
+	8950 5100 9050 5100
 Text Label 3300 5000 0    50   ~ 0
 ResultAdc
@@
 	3300 5000 3200 5000
 Connection ~ 3200 5000
-Text Label 9850 5150 2    50   ~ 0
+Text Label 8950 5200 2    50   ~ 0
 SourceAPwm
-Text Label 9850 5250 2    50   ~ 0
+Text Label 8950 5300 2    50   ~ 0
 SourceAAdc
-Text Label 9850 5350 2    50   ~ 0
+Text Label 8950 5400 2    50   ~ 0
 SourceBPwm
-Text Label 9850 5450 2    50   ~ 0
+Text Label 8950 5500 2    50   ~ 0
 SourceBAdc
-Text Label 9850 5550 2    50   ~ 0
+Text Label 8950 5600 2    50   ~ 0
 ResultAdc
 Wire Wire Line
-	9850 5150 9950 5150
-Wire Wire Line
-	9850 5250 9950 5250
-Wire Wire Line
-	9850 5350 9950 5350
-Wire Wire Line
-	9850 5450 9950 5450
-Wire Wire Line
-	9850 5550 9950 5550
+	8950 5200 9050 5200
+Wire Wire Line
+	8950 5300 9050 5300
+Wire Wire Line
+	8950 5400 9050 5400
+Wire Wire Line
+	8950 5500 9050 5500
+Wire Wire Line
+	8950 5600 9050 5600
 $Comp
 L Connector_Generic:Conn_01x15 J3
 U 1 1 6212FC4C
-P 10150 5250
-F 0 "J3" H 10230 5292 50  0000 L CNN
-F 1 "Conn_01x15" H 10230 5201 50  0000 L CNN
-F 2 "Connector_PinSocket_2.54mm:PinSocket_1x15_P2.54mm_Vertical" H 10150 5250 50  0001 C CNN
-F 3 "~" H 10150 5250 50  0001 C CNN
-F 4 "Do Not Fit" H 10150 5250 50  0001 C CNN "Vendor"
-	1    10150 5250
+P 9250 5300
+F 0 "J3" H 9330 5342 50  0000 L CNN
+F 1 "Conn_01x15" H 9330 5251 50  0000 L CNN
+F 2 "Connector_PinSocket_2.54mm:PinSocket_1x15_P2.54mm_Vertical" H 9250 5300 50  0001 C CNN
+F 3 "~" H 9250 5300 50  0001 C CNN
+F 4 "Do Not Fit" H 9250 5300 50  0001 C CNN "Vendor"
+	1    9250 5300
 	1    0    0    -1
 $EndComp
@@
 L power:+5V #PWR012
 U 1 1 62001D6A
-P 9200 5550
-F 0 "#PWR012" H 9200 5400 50  0001 C CNN
-F 1 "+5V" H 9215 5723 50  0000 C CNN
-F 2 "" H 9200 5550 50  0001 C CNN
-F 3 "~" H 9200 5550 50  0001 C CNN
-	1    9200 5550
-	1    0    0    -1
-$EndComp
-Wire Wire Line
-	9200 5550 9200 5650
-Wire Wire Line
-	9200 5650 9200 5750
-Connection ~ 9200 5650
+P 8300 5600
+F 0 "#PWR012" H 8300 5450 50  0001 C CNN
+F 1 "+5V" H 8315 5773 50  0000 C CNN
+F 2 "" H 8300 5600 50  0001 C CNN
+F 3 "~" H 8300 5600 50  0001 C CNN
+	1    8300 5600
+	1    0    0    -1
+$EndComp
+Wire Wire Line
+	8300 5600 8300 5700
+Wire Wire Line
+	8300 5700 8300 5800
+Connection ~ 8300 5700
 $Comp
 L power:GND #PWR013
 U 1 1 62050EDB
-P 9200 6050
-F 0 "#PWR013" H 9200 5800 50  0001 C CNN
-F 1 "GND" H 9205 5877 50  0000 C CNN
-F 2 "" H 9200 6050 50  0001 C CNN
-F 3 "~" H 9200 6050 50  0001 C CNN
-	1    9200 6050
-	1    0    0    -1
-$EndComp
-Wire Wire Line
-	9200 5850 9200 5950
-Wire Wire Line
-	9200 5950 9200 6050
-Connection ~ 9200 5950
-Wire Wire Line
-	9200 5650 9950 5650
-Wire Wire Line
-	9200 5750 9950 5750
-Wire Wire Line
-	9200 5850 9950 5850
-Wire Wire Line
-	9200 5950 9950 5950
+P 8300 6100
+F 0 "#PWR013" H 8300 5850 50  0001 C CNN
+F 1 "GND" H 8305 5927 50  0000 C CNN
+F 2 "" H 8300 6100 50  0001 C CNN
+F 3 "~" H 8300 6100 50  0001 C CNN
+	1    8300 6100
+	1    0    0    -1
+$EndComp
+Wire Wire Line
+	8300 5900 8300 6000
+Wire Wire Line
+	8300 6000 8300 6100
+Connection ~ 8300 6000
+Wire Wire Line
+	8300 5700 9050 5700
+Wire Wire Line
+	8300 5800 9050 5800
+Wire Wire Line
+	8300 5900 9050 5900
+Wire Wire Line
+	8300 6000 9050 6000
 $Comp
 L Device:R R14
@@
 $EndComp
 $Comp
-L Device:CP1 C?
+L Device:CP1 C10
 U 1 1 62175534
 P 7850 3900
-F 0 "C?" H 7965 3946 50  0000 L CNN
+F 0 "C10" H 7965 3946 50  0000 L CNN
 F 1 "5uF" H 7965 3855 50  0000 L CNN
 F 2 "" H 7850 3900 50  0001 C CNN
@@
 Determine\ncombination\nwith testing
 $Comp
-L Device:CP1 C?
+L Device:CP1 C9
 U 1 1 621C95BD
 P 7800 1750
-F 0 "C?" H 7915 1796 50  0000 L CNN
+F 0 "C9" H 7915 1796 50  0000 L CNN
 F 1 "5uF" H 7915 1705 50  0000 L CNN
 F 2 "" H 7800 1750 50  0001 C CNN
@@
 	6850 1600 8150 1600
 $Comp
-L amper-symbols:ATtiny1606-S U?
+L amper-symbols:ATtiny1606-S U6
 U 1 1 62224E78
 P 9700 3150
-F 0 "U?" H 9700 4115 50  0000 C CNN
+F 0 "U6" H 9700 4115 50  0000 C CNN
 F 1 "ATtiny1606-S" H 9700 4024 50  0000 C CNN
 F 2 "Package_SO:SOIC-20W_7.5x12.8mm_P1.27mm" H 9700 2800 50  0001 C CIN
@@
 	10300 2450 10400 2450
 $Comp
-L power:+5V #PWR?
+L power:+5V #PWR0101
 U 1 1 622DD6E8
 P 9000 2350
-F 0 "#PWR?" H 9000 2200 50  0001 C CNN
+F 0 "#PWR0101" H 9000 2200 50  0001 C CNN
 F 1 "+5V" H 9015 2523 50  0000 C CNN
 F 2 "" H 9000 2350 50  0001 C CNN
@@
 	9000 2450 9100 2450
 $Comp
-L power:GND #PWR?
+L power:GND #PWR0102
 U 1 1 622EC3F9
 P 10150 2100
-F 0 "#PWR?" H 10150 1850 50  0001 C CNN
+F 0 "#PWR0102" H 10150 1850 50  0001 C CNN
 F 1 "GND" H 10155 1927 50  0000 C CNN
 F 2 "" H 10150 2100 50  0001 C CNN
@@
 Text Label 10350 2950 0    50   ~ 0
 SourceBDn
+$Comp
+L Connector_Generic:Conn_01x03 J6
+U 1 1 62424A8C
+P 11000 4000
+F 0 "J6" H 11000 4300 50  0000 C CNN
+F 1 "Conn_01x03" H 11000 4200 50  0000 C CNN
+F 2 "amper:PROG" H 11000 4000 50  0001 C CNN
+F 3 "~" H 11000 4000 50  0001 C CNN
+	1    11000 4000
+	1    0    0    -1
+$EndComp
+$Comp
+L Connector_Generic:Conn_01x04 J7
+U 1 1 624255C1
+P 11000 4950
+F 0 "J7" H 11000 5250 50  0000 C CNN
+F 1 "Conn_01x04" H 11000 5150 50  0000 C CNN
+F 2 "amper:UART" H 11000 4950 50  0001 C CNN
+F 3 "~" H 11000 4950 50  0001 C CNN
+	1    11000 4950
+	1    0    0    -1
+$EndComp
+$Comp
+L power:+5V #PWR0103
+U 1 1 6242928C
+P 10700 3800
+F 0 "#PWR0103" H 10700 3650 50  0001 C CNN
+F 1 "+5V" H 10715 3973 50  0000 C CNN
+F 2 "" H 10700 3800 50  0001 C CNN
+F 3 "" H 10700 3800 50  0001 C CNN
+	1    10700 3800
+	1    0    0    -1
+$EndComp
+Wire Wire Line
+	10700 3800 10700 3900
+Wire Wire Line
+	10700 3900 10800 3900
+$Comp
+L power:GND #PWR0104
+U 1 1 6243649F
+P 10700 4200
+F 0 "#PWR0104" H 10700 3950 50  0001 C CNN
+F 1 "GND" H 10705 4027 50  0000 C CNN
+F 2 "" H 10700 4200 50  0001 C CNN
+F 3 "" H 10700 4200 50  0001 C CNN
+	1    10700 4200
+	1    0    0    -1
+$EndComp
+Wire Wire Line
+	10700 4200 10700 4100
+Wire Wire Line
+	10700 4100 10800 4100
+Text Label 10700 4000 2    50   ~ 0
+AtProg
+Wire Wire Line
+	10700 4000 10800 4000
+$Comp
+L power:+5V #PWR0105
+U 1 1 62454C28
+P 10700 4750
+F 0 "#PWR0105" H 10700 4600 50  0001 C CNN
+F 1 "+5V" H 10715 4923 50  0000 C CNN
+F 2 "" H 10700 4750 50  0001 C CNN
+F 3 "" H 10700 4750 50  0001 C CNN
+	1    10700 4750
+	1    0    0    -1
+$EndComp
+Wire Wire Line
+	10700 4750 10700 4850
+Wire Wire Line
+	10700 4850 10800 4850
+$Comp
+L power:GND #PWR0106
+U 1 1 62454C30
+P 10700 5250
+F 0 "#PWR0106" H 10700 5000 50  0001 C CNN
+F 1 "GND" H 10705 5077 50  0000 C CNN
+F 2 "" H 10700 5250 50  0001 C CNN
+F 3 "" H 10700 5250 50  0001 C CNN
+	1    10700 5250
+	1    0    0    -1
+$EndComp
+Wire Wire Line
+	10700 5250 10700 5150
+Wire Wire Line
+	10700 5150 10800 5150
+Text Label 10700 4950 2    50   ~ 0
+UartTx
+Wire Wire Line
+	10700 4950 10800 4950
+Text Label 10700 5050 2    50   ~ 0
+UartRx
+Wire Wire Line
+	10700 5050 10800 5050
 $EndSCHEMATC

Commit message: fixed library
Parts:
- removed J3: Conn_01x15, Connector_PinSocket_2.54mm:PinSocket_1x15_P2.54mm_Vertical, symbol Connector_Generic:Conn_01x15
- removed J4, J5: Conn_01x10, Connector_PinSocket_2.54mm:PinSocket_1x10_P2.54mm_Vertical, symbol Connector_Generic:Conn_01x10
Connections:
- net SourceAAdc renamed SourceAOut
- net SourceBAdc renamed SourceBOut
- no-connect marks 11 -> 15
Other:
- note added: "Expose these traces\nfor ease of bodging"
- moved on the sheet: J6, J7, U6
